File: tracker/hardware/pico/pecanpico10.kicad_pcb (KiCad board)
At the start: 2 copper layers, 23 x 50 mm, 123 parts, among them IC1 SPV1040T, IC10 AS213, IC2 TPS62260DRVR, IC3 ADP322ACPZ-115-R7, IC4 Si4464-B1B-FM, IC5 STM32F413xG, IC6 EVA-7M, IC7 PAC1720-1-AIA-TR, IC8 TPS62260DRVR, IC9 BME280, J1 Micro_SD_Card_Det, J2 CONN_01X15, P1 CONN_01X25, P3 ZX62-B-5PA(33), P4 SMA, Q1 FDN306P, X1 KT2016K26000BCW18ZAS

Commit message: Modified component values, created BOM
Parts:
- AE1: value GPS-Antenna -> 1575AT43A0040E
- C26: value 22p -> 15p
- C27: value 3.3p -> N/A
- C49: value 3.3p -> 2.2p
- IC10: value AS213 -> AS213-92LF
- IC5: value STM32F413xG -> STM32F413RHT6
- IC6: value EVA-7M -> EVA-7M or EVA-M8
- J1: value Micro_SD_Card_Det -> DM3AT-SF-PEJM5
- L6: value 56n -> 0R
- L9: value 82n -> 56n
- R11: value 1k5 -> 1k
- R12: value 510k -> 470k
- R13: value 110k -> 100k
- R14, R9: value 100k -> 10k
- R7: value 510k -> 402k
- R8: value 250k -> 100k
Changed lines of the file:
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@@
     (links 404)
     (no_connects 0)
-    (area -9.573976 63.201725 76.900001 127.750001)
+    (area 47.049999 74.549999 70.150001 124.650001)
     (thickness 1)
     (drawings 28)
@@
       (effects (font (size 1 1) (thickness 0.15)) (justify mirror))
     )
-    (fp_text value Micro_SD_Card_Det (at -2.85 -16.7 180) (layer B.Fab) hide
+    (fp_text value DM3AT-SF-PEJM5 (at -2.85 -16.7 180) (layer B.Fab) hide
       (effects (font (size 1 1) (thickness 0.15)) (justify mirror))
     )
@@
       (effects (font (size 1 1) (thickness 0.15)))
     )
-    (fp_text value STM32F413xG (at 0 7.2) (layer F.Fab)
+    (fp_text value STM32F413RHT6 (at 0 7.2) (layer F.Fab)
       (effects (font (size 1 1) (thickness 0.15)))
     )
@@
       (effects (font (size 0.5 0.5) (thickness 0.075)))
     )
-    (fp_text value EVA-7M (at 0 2.3 180) (layer F.Fab) hide
+    (fp_text value "EVA-7M or EVA-M8" (at 0 2.3 180) (layer F.Fab) hide
       (effects (font (size 0.5 0.5) (thickness 0.075)))
     )
@@
       (effects (font (size 0.127 0.127) (thickness 0.01875)))
     )
-    (fp_text value 22p (at 0.1 0 180) (layer F.Fab)
+    (fp_text value 15p (at 0.1 0 180) (layer F.Fab)
       (effects (font (size 0.127 0.127) (thickness 0.015875)))
     )
@@
       (effects (font (size 0.127 0.127) (thickness 0.01875)))
     )
-    (fp_text value 3.3p (at 0.1 0 180) (layer F.Fab)
+    (fp_text value N/A (at 0.1 0 180) (layer F.Fab)
       (effects (font (size 0.127 0.127) (thickness 0.015875)))
     )
@@
       (effects (font (size 0.127 0.127) (thickness 0.01875)))
     )
-    (fp_text value 510k (at 0.1 0 90) (layer F.Fab)
+    (fp_text value 402k (at 0.1 0 90) (layer F.Fab)
       (effects (font (size 0.127 0.127) (thickness 0.01875)))
     )
@@
       (effects (font (size 0.127 0.127) (thickness 0.01875)))
     )
-    (fp_text value 250k (at 0.1 0 90) (layer F.Fab)
+    (fp_text value 100k (at 0.1 0 90) (layer F.Fab)
       (effects (font (size 0.127 0.127) (thickness 0.01875)))
     )
@@
       (effects (font (size 0.127 0.127) (thickness 0.01875)))
     )
-    (fp_text value 100k (at 0.1 0 180) (layer F.Fab)
+    (fp_text value 10k (at 0.1 0 180) (layer F.Fab)
       (effects (font (size 0.127 0.127) (thickness 0.01875)))
     )
@@
       (effects (font (size 0.127 0.127) (thickness 0.01875)))
     )
-    (fp_text value 1k5 (at 0.1 0 360) (layer F.Fab)
+    (fp_text value 1k (at 0.1 0 360) (layer F.Fab)
       (effects (font (size 0.127 0.127) (thickness 0.01875)))
     )
@@
       (effects (font (size 0.127 0.127) (thickness 0.01875)))
     )
-    (fp_text value 100k (at 0.1 0 270) (layer F.Fab)
+    (fp_text value 10k (at 0.1 0 270) (layer F.Fab)
       (effects (font (size 0.127 0.127) (thickness 0.01875)))
     )
@@
       (effects (font (size 0.127 0.127) (thickness 0.01875)))
     )
-    (fp_text value 510k (at 0.1 0 90) (layer F.Fab)
+    (fp_text value 470k (at 0.1 0 90) (layer F.Fab)
       (effects (font (size 0.127 0.127) (thickness 0.01875)))
     )
@@
       (effects (font (size 0.127 0.127) (thickness 0.01875)))
     )
-    (fp_text value 110k (at 0.1 0 90) (layer F.Fab)
+    (fp_text value 100k (at 0.1 0 90) (layer F.Fab)
       (effects (font (size 0.127 0.127) (thickness 0.01875)))
     )
@@
       (effects (font (size 0.127 0.127) (thickness 0.01875)))
     )
-    (fp_text value 3.3p (at 0.1 0 180) (layer F.Fab)
+    (fp_text value 2.2p (at 0.1 0 180) (layer F.Fab)
       (effects (font (size 0.127 0.127) (thickness 0.015875)))
     )
@@
       (effects (font (size 0.166 0.166) (thickness 0.025)))
     )
-    (fp_text value 82n (at 0.2 0 360) (layer F.Fab)
+    (fp_text value 56n (at 0.2 0 360) (layer F.Fab)
       (effects (font (size 0.166 0.166) (thickness 0.025)))
     )
@@
       (effects (font (size 0.166 0.166) (thickness 0.025)))
     )
-    (fp_text value 56n (at 0.2 0 360) (layer F.Fab)
+    (fp_text value 0R (at 0.2 0 360) (layer F.Fab)
       (effects (font (size 0.166 0.166) (thickness 0.025)))
     )
@@
       (effects (font (size 0.25 0.25) (thickness 0.0375)))
     )
-    (fp_text value GPS-Antenna (at 0.75 0 270) (layer F.Fab)
+    (fp_text value 1575AT43A0040E (at 0.75 0 270) (layer F.Fab)
       (effects (font (size 0.25 0.25) (thickness 0.0375)))
     )
@@
       (effects (font (size 0.25 0.25) (thickness 0.0375)))
     )
-    (fp_text value AS213 (at 1.8 0 90) (layer F.Fab) hide
+    (fp_text value AS213-92LF (at 1.8 0 90) (layer F.Fab) hide
       (effects (font (size 0.25 0.25) (thickness 0.0375)))
     )
